Commit message: Task N stuck

File: body.urdf (robot description, URDF)
Before this commit: robot robot, 3 links, 2 joints
Links:
- added link BackLowerLeg, mass 1; collision box size=0.2 0.2 1; visual box size=0.2 0.2 1
- added link FrontLowerLeg, mass 1; collision box size=0.2 0.2 1; visual box size=0.2 0.2 1
- added link LeftLeg, mass 1; collision box size=1 0.2 0.2; visual box size=1 0.2 0.2
- added link LeftLowerLeg, mass 1; collision box size=0.2 0.2 1; visual box size=0.2 0.2 1
- added link RightLeg, mass 1; collision box size=1 0.2 0.2; visual box size=1 0.2 0.2
- added link RightLowerLeg, mass 1; collision box size=0.2 0.2 1; visual box size=0.2 0.2 1
Joints:
- added joint BackLeg_BackLowerLeg: type revolute, parent BackLeg, child BackLowerLeg, origin xyz=0 -1 0 rpy=0 0 0, axis 1 0 0, limit lower=-3.14159 upper=3.14159 effort=0.0 velocity=0.0
- added joint FrontLeg_FrontLowerLeg: type revolute, parent FrontLeg, child FrontLowerLeg, origin xyz=0 1 0 rpy=0 0 0, axis 1 0 0, limit lower=-3.14159 upper=3.14159 effort=0.0 velocity=0.0
- added joint LeftLeg_LeftLowerLeg: type revolute, parent LeftLeg, child LeftLowerLeg, origin xyz=-1 0 0 rpy=0 0 0, axis 0 1 0, limit lower=-3.14159 upper=3.14159 effort=0.0 velocity=0.0
- added joint RightLeg_RightLowerLeg: type revolute, parent RightLeg, child RightLowerLeg, origin xyz=1 0 0 rpy=0 0 0, axis 0 1 0, limit lower=-3.14159 upper=3.14159 effort=0.0 velocity=0.0
- added joint Torso_LeftLeg: type revolute, parent Torso, child LeftLeg, origin xyz=-0.5 0 1 rpy=0 0 0, axis 0 1 0, limit lower=-3.14159 upper=3.14159 effort=0.0 velocity=0.0
- added joint Torso_RightLeg: type revolute, parent Torso, child RightLeg, origin xyz=0.5 0 1 rpy=0 0 0, axis 0 1 0, limit lower=-3.14159 upper=3.14159 effort=0.0 velocity=0.0

Commit message: Final

File: body.urdf (robot description, URDF)
Before this commit: robot robot, 9 links, 8 joints
Links:
- removed link BackLeg
- removed link BackLowerLeg
- removed link FrontLeg
- removed link FrontLowerLeg
- removed link LeftLeg
- removed link RightLeg
- added link BackLegLeft, mass 1; collision box size=0.2 0.3 0.1; visual box size=0.2 0.3 0.1
- added link BackLegRight, mass 1; collision box size=0.2 0.3 0.1; visual box size=0.2 0.3 0.1
- added link FrontLegLeft, mass 1; collision box size=0.2 0.3 0.1; visual box size=0.2 0.3 0.1
- added link FrontLegRight, mass 1; collision box size=0.2 0.3 0.1; visual box size=0.2 0.3 0.1
- added link LBLowerLeg, mass 1; collision box size=0.2 0.2 1; visual box size=0.2 0.2 1
- added link LFLowerLeg, mass 1; collision box size=0.2 0.2 1; visual box size=0.2 0.2 1
- added link LeftWing, mass 1; collision box size=0.2 0.2 0.1; visual box size=0.2 0.2 0.1
- added link RBLowerLeg, mass 1; collision box size=0.2 0.2 1; visual box size=0.2 0.2 1
- added link RFLowerLeg, mass 1; collision box size=0.2 0.2 1; visual box size=0.2 0.2 1
- added link RightWing, mass 1; collision box size=0.2 0.2 0.1; visual box size=0.2 0.2 0.1
- link LeftLowerLeg: geometry collision box size=1.5 2 0.1; visual box size=1.5 2 0.1
- link RightLowerLeg: geometry collision box size=1.5 2 0.1; visual box size=1.5 2 0.1
- link Torso: geometry collision box size=3 0.7 0.4; visual box size=3 0.7 0.4
Joints:
- removed joint BackLeg_BackLowerLeg
- removed joint FrontLeg_FrontLowerLeg
- removed joint LeftLeg_LeftLowerLeg
- removed joint RightLeg_RightLowerLeg
- removed joint Torso_BackLeg
- removed joint Torso_FrontLeg
- removed joint Torso_LeftLeg
- removed joint Torso_RightLeg
- added joint BackLegLeft_LBLowerLeg: type revolute, parent BackLegLeft, child LBLowerLeg, origin xyz=0 0.3 0 rpy=0 0 0, axis 0 1 0, limit lower=-3.14159 upper=3.14159 effort=0.0 velocity=0.0
- added joint BackLegRight_RBLowerLeg: type revolute, parent BackLegRight, child RBLowerLeg, origin xyz=0 -0.3 0 rpy=0 0 0, axis 0 1 0, limit lower=-3.14159 upper=3.14159 effort=0.0 velocity=0.0
- added joint FrontLegLeft_LFLowerLeg: type revolute, parent FrontLegLeft, child LFLowerLeg, origin xyz=0 0.3 0 rpy=0 0 0, axis 0 1 0, limit lower=-3.14159 upper=3.14159 effort=0.0 velocity=0.0
- added joint FrontLegRight_RFLowerLeg: type revolute, parent FrontLegRight, child RFLowerLeg, origin xyz=0 -0.3 0 rpy=0 0 0, axis 0 1 0, limit lower=-3.14159 upper=3.14159 effort=0.0 velocity=0.0
- added joint LeftWing_LeftLowerLeg: type revolute, parent LeftWing, child LeftLowerLeg, origin xyz=0 0.1 0 rpy=0 0 0, axis 1 0 0, limit lower=-3.14159 upper=3.14159 effort=0.0 velocity=0.0
- added joint RightWing_RightLowerLeg: type revolute, parent RightWing, child RightLowerLeg, origin xyz=0 -0.1 0 rpy=0 0 0, axis 1 0 0, limit lower=-3.14159 upper=3.14159 effort=0.0 velocity=0.0
- added joint Torso_BackLegLeft: type revolute, parent Torso, child BackLegLeft, origin xyz=-1.05 0.35 3 rpy=0 0 0, axis 1 0 0, limit lower=-3.14159 upper=3.14159 effort=0.0 velocity=0.0
- added joint Torso_BackLegRight: type revolute, parent Torso, child BackLegRight, origin xyz=-1.05 -0.35 3 rpy=0 0 0, axis 1 0 0, limit lower=-3.14159 upper=3.14159 effort=0.0 velocity=0.0
- added joint Torso_FrontLegLeft: type revolute, parent Torso, child FrontLegLeft, origin xyz=1.05 0.35 3 rpy=0 0 0, axis 1 0 0, limit lower=-3.14159 upper=3.14159 effort=0.0 velocity=0.0
- added joint Torso_FrontLegRight: type revolute, parent Torso, child FrontLegRight, origin xyz=1.05 -0.35 3 rpy=0 0 0, axis 1 0 0, limit lower=-3.14159 upper=3.14159 effort=0.0 velocity=0.0
- added joint Torso_LeftWing: type revolute, parent Torso, child LeftWing, origin xyz=0 0.35 3 rpy=0 0 0, axis 1 0 0, limit lower=-3.14159 upper=3.14159 effort=0.0 velocity=0.0
- added joint Torso_RightWing: type revolute, parent Torso, child RightWing, origin xyz=0 -0.35 3 rpy=0 0 0, axis 1 0 0, limit lower=-3.14159 upper=3.14159 effort=0.0 velocity=0.0

Commit message: Without color change

File: body.urdf (robot description, URDF)
Before this commit: robot robot, 13 links, 12 joints
Links:
- removed link BackLegLeft
- removed link BackLegRight
- removed link FrontLegLeft
- removed link FrontLegRight
- removed link LBLowerLeg
- removed link LFLowerLeg
- removed link LeftLowerLeg
- removed link LeftWing
- removed link RBLowerLeg
- removed link RFLowerLeg
- removed link RightLowerLeg
- removed link RightWing
- removed link Torso
- added link Link0, mass 1; collision box size=0.31128868730713954 0.009844703597124638 0.25127639220033127; visual box size=0.31128868730713954 0.009844703597124638 0.25127639220033127
- added link Link1, mass 1; collision box size=1.656166769163059 0.9858934662567198 0.25127639220033127; visual box size=1.656166769163059 0.9858934662567198 0.25127639220033127
- added link Link2, mass 1; collision box size=0.2418077504858298 1.0551022045272562 0.25127639220033127; visual box size=0.2418077504858298 1.0551022045272562 0.25127639220033127
Joints:
- removed joint BackLegLeft_LBLowerLeg
- removed joint BackLegRight_RBLowerLeg
- removed joint FrontLegLeft_LFLowerLeg
- removed joint FrontLegRight_RFLowerLeg
- removed joint LeftWing_LeftLowerLeg
- removed joint RightWing_RightLowerLeg
- removed joint Torso_BackLegLeft
- removed joint Torso_BackLegRight
- removed joint Torso_FrontLegLeft
- removed joint Torso_FrontLegRight
- removed joint Torso_LeftWing
- removed joint Torso_RightWing
- added joint Link0_Link1: type revolute, parent Link0, child Link1, origin xyz=0.15564434365356977 0 0 rpy=0 0 0, axis 0 0 1, limit lower=-3.14159 upper=3.14159 effort=0.0 velocity=0.0
- added joint Link1_Link2: type revolute, parent Link1, child Link2, origin xyz=1.656166769163059 0 0 rpy=0 0 0, axis 0 0 1, limit lower=-3.14159 upper=3.14159 effort=0.0 velocity=0.0

Commit message: Snake color resolved

File: body.urdf (robot description, URDF)
Before this commit: robot robot, 3 links, 2 joints
Links:
- added link Link3, mass 1; collision box size=0.926087290339999 0.7887750014393143 0.16150675628798372; visual box size=0.926087290339999 0.7887750014393143 0.16150675628798372
- added link Link4, mass 1; collision box size=0.4478657431777756 0.8322603039506715 0.16150675628798372; visual box size=0.4478657431777756 0.8322603039506715 0.16150675628798372
- added link Link5, mass 1; collision box size=0.3159197498960473 0.9743832551064457 0.16150675628798372; visual box size=0.3159197498960473 0.9743832551064457 0.16150675628798372
- added link Link6, mass 1; collision box size=2.422287169561697 0.3758904370902476 0.16150675628798372; visual box size=2.422287169561697 0.3758904370902476 0.16150675628798372
- added link Link7, mass 1; collision box size=0.28671540833622433 0.4784751442878553 0.16150675628798372; visual box size=0.28671540833622433 0.4784751442878553 0.16150675628798372
- link Link0: geometry collision box size=0.8278357671955487 1.2369030982280245 3; visual box size=0.8278357671955487 1.2369030982280245 3
- link Link1: geometry collision box size=0.5140031015249679 1.7005796065996661 0.16150675628798372; visual box size=0.5140031015249679 1.7005796065996661 0.16150675628798372
- link Link2: geometry collision box size=0.09104046702848212 1.1309116987738974 0.16150675628798372; visual box size=0.09104046702848212 1.1309116987738974 0.16150675628798372
Joints:
- added joint Link2_Link3: type revolute, parent Link2, child Link3, origin xyz=0.04552023351424106 0 0 rpy=0 0 0, axis 0 0 1, limit lower=-3.14159 upper=3.14159 effort=0.0 velocity=0.0
- added joint Link3_Link4: type revolute, parent Link3, child Link4, origin xyz=0.4630436451699995 0 0 rpy=0 0 0, axis 0 0 1, limit lower=-3.14159 upper=3.14159 effort=0.0 velocity=0.0
- added joint Link4_Link5: type revolute, parent Link4, child Link5, origin xyz=0.2239328715888878 0 0 rpy=0 0 0, axis 0 0 1, limit lower=-3.14159 upper=3.14159 effort=0.0 velocity=0.0
- added joint Link5_Link6: type revolute, parent Link5, child Link6, origin xyz=0.15795987494802366 0 0 rpy=0 0 0, axis 0 0 1, limit lower=-3.14159 upper=3.14159 effort=0.0 velocity=0.0
- added joint Link6_Link7: type revolute, parent Link6, child Link7, origin xyz=1.2111435847808485 0 0 rpy=0 0 0, axis 0 0 1, limit lower=-3.14159 upper=3.14159 effort=0.0 velocity=0.0
- joint Link0_Link1: origin xyz=0.15564434365356977 0 0 rpy=0 0 0 -> xyz=0.41391788359777437 0 3 rpy=0 0 0
- joint Link1_Link2: origin xyz=1.656166769163059 0 0 rpy=0 0 0 -> xyz=0.25700155076248393 0 0 rpy=0 0 0

Commit message: Snakes Complete

File: body.urdf (robot description, URDF)
Before this commit: robot robot, 8 links, 7 joints
Links:
- removed link Link4
- removed link Link5
- removed link Link6
- removed link Link7
- link Link0: geometry collision box size=0.03673619997716404 0.41113029052463546 2; visual box size=0.03673619997716404 0.41113029052463546 2
- link Link1: geometry collision box size=0.8635453016144459 0.5143596462778961 0.13089836352824924; visual box size=0.8635453016144459 0.5143596462778961 0.13089836352824924
- link Link2: geometry collision box size=0.3716243297303228 0.6663487557258075 0.13089836352824924; visual box size=0.3716243297303228 0.6663487557258075 0.13089836352824924
- link Link3: geometry collision box size=0.43667157318844907 0.9269817520927305 0.13089836352824924; visual box size=0.43667157318844907 0.9269817520927305 0.13089836352824924
Joints:
- removed joint Link3_Link4
- removed joint Link4_Link5
- removed joint Link5_Link6
- removed joint Link6_Link7
- joint Link0_Link1: origin xyz=0.41391788359777437 0 3 rpy=0 0 0 -> xyz=0.01836809998858202 0 1 rpy=0 0 0
- joint Link1_Link2: origin xyz=0.25700155076248393 0 0 rpy=0 0 0 -> xyz=0.8635453016144459 0 0 rpy=0 0 0
- joint Link2_Link3: origin xyz=0.04552023351424106 0 0 rpy=0 0 0 -> xyz=0.3716243297303228 0 0 rpy=0 0 0

Commit message: Left a bit

File: body.urdf (robot description, URDF)
Before this commit: robot robot, 9 links, 8 joints
Links:
- removed link Link3
- removed link Link4
- removed link Link5
- removed link Link6
- removed link Link7
- removed link Link8
- link Link0: geometry collision box size=1 1 2; visual box size=1 1 2
- link Link1: geometry collision box size=1 2 1; visual box size=1 2 1
- link Link2: geometry collision box size=1 2 2; visual box size=1 2 2
Joints:
- removed joint Link0_Link3
- removed joint Link2_Link6
- removed joint Link3_Link4
- removed joint Link4_Link5
- removed joint Link6_Link7
- removed joint Link7_Link8
- joint Link0_Link1: origin xyz=0.5 0.5 1.5 rpy=0 0 0 -> xyz=0.5 0.5 2 rpy=0 0 0

Commit message: Almost

File: body.urdf (robot description, URDF)
Before this commit: robot robot, 3 links, 2 joints
Links:
- added link Link3, mass 1; collision box size=4 3 2; visual box size=4 3 2
- link Link0: geometry collision box size=3 4 1; visual box size=3 4 1
- link Link1: geometry collision box size=2 1 2; visual box size=2 1 2
- link Link2: geometry collision box size=1 3 1; visual box size=1 3 1
Joints:
- added joint Link1_Link3: type revolute, parent Link1, child Link3, origin xyz=1.0 0 1.0 rpy=0 0 0, axis 0 0 1, limit lower=-3.14159 upper=3.14159 effort=0.0 velocity=0.0
- joint Link0_Link1: axis 0 0 1 -> 1 0 0; origin xyz=0.5 0.5 2 rpy=0 0 0 -> xyz=3 2.0 0.5 rpy=0 0 0
- joint Link1_Link2: axis 0 0 1 -> 1 0 0; origin xyz=0 0 1 rpy=0 0 0 -> xyz=2 0 0 rpy=0 0 0

Commit message: completed

File: body.urdf (robot description, URDF)
Before this commit: robot robot, 4 links, 3 joints
Links:
- link Link0: geometry collision box size=2 1 2; visual box size=2 1 2
- link Link1: geometry collision box size=1 3 1; visual box size=1 3 1
- link Link2: geometry collision box size=4 1 1; visual box size=4 1 1
- link Link3: geometry collision box size=2 1 2; visual box size=2 1 2
Joints:
- removed joint Link1_Link2
- removed joint Link1_Link3
- added joint Link0_Link2: type revolute, parent Link0, child Link2, origin xyz=2 0.5 1.0 rpy=0 0 0, axis 1 0 0, limit lower=-3.14159 upper=3.14159 effort=0.0 velocity=0.0
- added joint Link0_Link3: type revolute, parent Link0, child Link3, origin xyz=1.0 1 1.0 rpy=0 0 0, axis 0 1 0, limit lower=-3.14159 upper=3.14159 effort=0.0 velocity=0.0
- joint Link0_Link1: axis 1 0 0 -> 0 0 1; origin xyz=3 2.0 0.5 rpy=0 0 0 -> xyz=1.0 0.5 2 rpy=0 0 0

Commit message: Value increased

File: body.urdf (robot description, URDF)
Before this commit: robot robot, 4 links, 3 joints
Links:
- added link Link10, mass 1; collision box size=1 2 2; visual box size=1 2 2
- added link Link11, mass 1; collision box size=3 3 2; visual box size=3 3 2
- added link Link4, mass 1; collision box size=3 4 2; visual box size=3 4 2
- added link Link5, mass 1; collision box size=4 1 1; visual box size=4 1 1
- added link Link6, mass 1; collision box size=1 1 1; visual box size=1 1 1
- added link Link7, mass 1; collision box size=3 3 2; visual box size=3 3 2
- added link Link8, mass 1; collision box size=1 2 2; visual box size=1 2 2
- added link Link9, mass 1; collision box size=3 3 1; visual box size=3 3 1
- link Link0: geometry collision box size=4 4 2; visual box size=4 4 2
- link Link1: geometry collision box size=4 4 2; visual box size=4 4 2
- link Link2: geometry collision box size=1 1 2; visual box size=1 1 2
- link Link3: geometry collision box size=1 3 1; visual box size=1 3 1
Joints:
- removed joint Link0_Link3
- added joint Link1_Link10: type revolute, parent Link1, child Link10, origin xyz=0 2.0 1.0 rpy=0 0 0, axis 0 0 1, limit lower=-3.14159 upper=3.14159 effort=0.0 velocity=0.0
- added joint Link1_Link3: type revolute, parent Link1, child Link3, origin xyz=0 4 0 rpy=0 0 0, axis 0 1 0, limit lower=-3.14159 upper=3.14159 effort=0.0 velocity=0.0
- added joint Link2_Link4: type revolute, parent Link2, child Link4, origin xyz=0 0.5 1.0 rpy=0 0 0, axis 0 1 0, limit lower=-3.14159 upper=3.14159 effort=0.0 velocity=0.0
- added joint Link3_Link5: type revolute, parent Link3, child Link5, origin xyz=0 3 0 rpy=0 0 0, axis 0 1 0, limit lower=-3.14159 upper=3.14159 effort=0.0 velocity=0.0
- added joint Link4_Link7: type revolute, parent Link4, child Link7, origin xyz=0 2.0 1.0 rpy=0 0 0, axis 0 0 1, limit lower=-3.14159 upper=3.14159 effort=0.0 velocity=0.0
- added joint Link5_Link11: type revolute, parent Link5, child Link11, origin xyz=0 0.5 0.5 rpy=0 0 0, axis 0 0 1, limit lower=-3.14159 upper=3.14159 effort=0.0 velocity=0.0
- added joint Link5_Link6: type revolute, parent Link5, child Link6, origin xyz=2.0 0.5 0 rpy=0 0 0, axis 1 0 0, limit lower=-3.14159 upper=3.14159 effort=0.0 velocity=0.0
- added joint Link6_Link8: type revolute, parent Link6, child Link8, origin xyz=0.5 0.5 0 rpy=0 0 0, axis 0 1 0, limit lower=-3.14159 upper=3.14159 effort=0.0 velocity=0.0
- added joint Link7_Link9: type revolute, parent Link7, child Link9, origin xyz=0 0 2 rpy=0 0 0, axis 0 0 1, limit lower=-3.14159 upper=3.14159 effort=0.0 velocity=0.0
- joint Link0_Link1: axis 0 0 1 -> 0 1 0; origin xyz=1.0 0.5 2 rpy=0 0 0 -> xyz=2.0 4 1.0 rpy=0 0 0
- joint Link0_Link2: axis 1 0 0 -> 0 0 1; origin xyz=2 0.5 1.0 rpy=0 0 0 -> xyz=2.0 2.0 2 rpy=0 0 0
